File: cloak-xt.kicad_pcb (KiCad board)
At the start: 2 copper layers, 289.7 x 98 mm, 156 parts, among them J1 JST, U1 STM32F072CBT6, U3 XC6206PxxxMR-Regulator_Linear

Commit message: Complete matrix and add Skyloong knob module
Parts:
- added ENC1: ROT_SKYLOONG_HS, PCM_marbastlib-various:ROT_SKYLOONG_HS-Switch, F.Cu at (66.9, 83.1)
- added ENC2: ROT_SKYLOONG_HS, PCM_marbastlib-various:ROT_SKYLOONG_HS-Switch, F.Cu at (338.4, 83.1)
- added Q1: Q_PMOS_GSD, Package_TO_SOT_SMD:SOT-23, F.Cu at (67.7, 92.6)
- added Q2: Q_PMOS_GSD, Package_TO_SOT_SMD:SOT-23, F.Cu at (340.8, 92.2)
- added R1: 10k, Resistor_SMD:R_0603_1608Metric, F.Cu at (73.3, 91.9)
- added R2: 10k, Resistor_SMD:R_0603_1608Metric, F.Cu at (334.4, 93.4)
- moved D14 5.08 mm to (345.5, 87.1)
- moved D1 4.76 mm to (74.9, 83.9)
Connections:
- D1 pad 1: unconnected-(D1-K-Pad1) -> ROW1
- D10 pad 1: unconnected-(D10-K-Pad1) -> ROW1
- D11 pad 1: unconnected-(D11-K-Pad1) -> ROW1
- D12 pad 1: unconnected-(D12-K-Pad1) -> ROW1
- D13 pad 1: unconnected-(D13-K-Pad1) -> ROW1
- D14 pad 1: unconnected-(D14-K-Pad1) -> ROW1
- D15 pad 1: unconnected-(D15-K-Pad1) -> ROW2
- D16 pad 1: unconnected-(D16-K-Pad1) -> ROW2
- D17 pad 1: unconnected-(D17-K-Pad1) -> ROW2
- D18 pad 1: unconnected-(D18-K-Pad1) -> ROW2
- D19 pad 1: unconnected-(D19-K-Pad1) -> ROW2
- D2 pad 1: unconnected-(D2-K-Pad1) -> ROW1
- D20 pad 1: unconnected-(D20-K-Pad1) -> ROW2
- D21 pad 1: unconnected-(D21-K-Pad1) -> ROW2
- D22 pad 1: unconnected-(D22-K-Pad1) -> ROW2
- D23 pad 1: unconnected-(D23-K-Pad1) -> ROW2
- D24 pad 1: unconnected-(D24-K-Pad1) -> ROW2
- D25 pad 1: unconnected-(D25-K-Pad1) -> ROW2
- D26 pad 1: unconnected-(D26-K-Pad1) -> ROW2
- D27 pad 1: unconnected-(D27-K-Pad1) -> ROW2
- D28 pad 1: unconnected-(D28-K-Pad1) -> ROW2
- D29 pad 1: unconnected-(D29-K-Pad1) -> ROW3
- D3 pad 1: unconnected-(D3-K-Pad1) -> ROW1
- D31 pad 1: unconnected-(D31-K-Pad1) -> ROW3
- D32 pad 1: unconnected-(D32-K-Pad1) -> ROW3
- D33 pad 1: unconnected-(D33-K-Pad1) -> ROW3
- D34 pad 1: unconnected-(D34-K-Pad1) -> ROW3
- D35 pad 1: unconnected-(D35-K-Pad1) -> ROW3
- D36 pad 1: unconnected-(D36-K-Pad1) -> ROW3
- D37 pad 1: unconnected-(D37-K-Pad1) -> ROW3
- D38 pad 1: unconnected-(D38-K-Pad1) -> ROW3
- D39 pad 1: unconnected-(D39-K-Pad1) -> ROW3
- D4 pad 1: unconnected-(D4-K-Pad1) -> ROW1
- D40 pad 1: unconnected-(D40-K-Pad1) -> ROW3
- D41 pad 1: unconnected-(D41-K-Pad1) -> ROW3
- D42 pad 1: unconnected-(D42-K-Pad1) -> ROW3
- D43 pad 1: unconnected-(D43-K-Pad1) -> ROW4
- D45 pad 1: unconnected-(D45-K-Pad1) -> ROW4
- D46 pad 1: unconnected-(D46-K-Pad1) -> ROW4
- D47 pad 1: unconnected-(D47-K-Pad1) -> ROW4
- D48 pad 1: unconnected-(D48-K-Pad1) -> ROW4
- D49 pad 1: unconnected-(D49-K-Pad1) -> ROW4
- D5 pad 1: unconnected-(D5-K-Pad1) -> ROW1
- D50 pad 1: unconnected-(D50-K-Pad1) -> ROW4
- D51 pad 1: unconnected-(D51-K-Pad1) -> ROW4
- D52 pad 1: unconnected-(D52-K-Pad1) -> ROW4
- D53 pad 1: unconnected-(D53-K-Pad1) -> ROW4
- D54 pad 1: unconnected-(D54-K-Pad1) -> ROW4
- D55 pad 1: unconnected-(D55-K-Pad1) -> ROW4
- D56 pad 1: unconnected-(D56-K-Pad1) -> ROW4
- D57 pad 1: unconnected-(D57-K-Pad1) -> ROW4
- D58 pad 1: unconnected-(D58-K-Pad1) -> ROW4
- D59 pad 1: unconnected-(D59-K-Pad1) -> ROW4
- D6 pad 1: unconnected-(D6-K-Pad1) -> ROW1
- D60 pad 1: unconnected-(D60-K-Pad1) -> ROW4
- D62 pad 1: unconnected-(D62-K-Pad1) -> ROW4
- D63 pad 1: unconnected-(D63-K-Pad1) -> ROW4
- D64 pad 1: unconnected-(D64-K-Pad1) -> ROW4
- D65 pad 1: unconnected-(D65-K-Pad1) -> ROW4
- D67 pad 1: unconnected-(D67-K-Pad1) -> ROW4
- D68 pad 1: unconnected-(D68-K-Pad1) -> ROW4
- D69 pad 1: unconnected-(D69-K-Pad1) -> ROW4
- D7 pad 1: unconnected-(D7-K-Pad1) -> ROW1
- D8 pad 1: unconnected-(D8-K-Pad1) -> ROW1
- D9 pad 1: unconnected-(D9-K-Pad1) -> ROW1
- MX1 pad 1: unconnected-(MX1-Pad1) -> COL1
- MX10 pad 1: unconnected-(MX10-Pad1) -> COL10
- MX11 pad 1: unconnected-(MX11-Pad1) -> COL11
- MX12 pad 1: unconnected-(MX12-Pad1) -> COL12
- MX13 pad 1: unconnected-(MX13-Pad1) -> COL13
- MX14 pad 1: unconnected-(MX14-Pad1) -> COL14
- MX15 pad 1: unconnected-(MX15-Pad1) -> COL1
- MX16 pad 1: unconnected-(MX16-Pad1) -> COL2
- MX17 pad 1: unconnected-(MX17-Pad1) -> COL3
- MX18 pad 1: unconnected-(MX18-Pad1) -> COL4
- MX19 pad 1: unconnected-(MX19-Pad1) -> COL5
- MX2 pad 1: unconnected-(MX2-Pad1) -> COL2
- MX20 pad 1: unconnected-(MX20-Pad1) -> COL6
- MX21 pad 1: unconnected-(MX21-Pad1) -> COL7
- MX22 pad 1: unconnected-(MX22-Pad1) -> COL8
- MX23 pad 1: unconnected-(MX23-Pad1) -> COL9
- MX24 pad 1: unconnected-(MX24-Pad1) -> COL10
- MX25 pad 1: unconnected-(MX25-Pad1) -> COL11
- MX26 pad 1: unconnected-(MX26-Pad1) -> COL12
- MX27 pad 1: unconnected-(MX27-Pad1) -> COL13
- MX28 pad 1: unconnected-(MX28-Pad1) -> COL14
- MX29 pad 1: unconnected-(MX29-Pad1) -> COL1
- MX3 pad 1: unconnected-(MX3-Pad1) -> COL3
- MX30 pad 1: unconnected-(MX30-Pad1) -> Net-(D29-A)
- MX30 pad 2: unconnected-(MX30-Pad2) -> COL1
- MX31 pad 1: unconnected-(MX31-Pad1) -> COL2
- MX32 pad 1: unconnected-(MX32-Pad1) -> COL3
- MX33 pad 1: unconnected-(MX33-Pad1) -> COL4
- MX34 pad 1: unconnected-(MX34-Pad1) -> COL5
- MX35 pad 1: unconnected-(MX35-Pad1) -> COL6
- MX36 pad 1: unconnected-(MX36-Pad1) -> COL7
- MX37 pad 1: unconnected-(MX37-Pad1) -> COL8
- MX38 pad 1: unconnected-(MX38-Pad1) -> COL9
- MX39 pad 1: unconnected-(MX39-Pad1) -> COL10
- MX4 pad 1: unconnected-(MX4-Pad1) -> COL4
- MX40 pad 1: unconnected-(MX40-Pad1) -> COL11
- MX41 pad 1: unconnected-(MX41-Pad1) -> COL13
- MX42 pad 1: unconnected-(MX42-Pad1) -> COL14
- MX43 pad 1: unconnected-(MX43-Pad1) -> Net-(D43-A)
- MX43 pad 2: unconnected-(MX43-Pad2) -> COL1
- MX44 pad 1: unconnected-(MX44-Pad1) -> COL1
- MX45 pad 1: unconnected-(MX45-Pad1) -> COL2
- MX46 pad 1: unconnected-(MX46-Pad1) -> COL3
- MX47 pad 1: unconnected-(MX47-Pad1) -> COL4
- MX48 pad 1: unconnected-(MX48-Pad1) -> COL5
- MX49 pad 1: unconnected-(MX49-Pad1) -> COL6
- MX5 pad 1: unconnected-(MX5-Pad1) -> COL5
- MX50 pad 1: unconnected-(MX50-Pad1) -> COL7
- MX51 pad 1: unconnected-(MX51-Pad1) -> COL8
- MX52 pad 1: unconnected-(MX52-Pad1) -> COL9
- MX53 pad 1: unconnected-(MX53-Pad1) -> COL10
- MX54 pad 1: unconnected-(MX54-Pad1) -> COL11
- MX55 pad 1: unconnected-(MX55-Pad1) -> COL12
- MX56 pad 1: unconnected-(MX56-Pad1) -> COL13
- MX57 pad 1: unconnected-(MX57-Pad1) -> COL14
- MX58 pad 1: unconnected-(MX58-Pad1) -> COL1
- MX59 pad 1: unconnected-(MX59-Pad1) -> COL2
- MX6 pad 1: unconnected-(MX6-Pad1) -> COL6
- MX60 pad 1: unconnected-(MX60-Pad1) -> COL3
- MX61 pad 1: unconnected-(MX61-Pad1) -> Net-(D60-A)
- MX61 pad 2: unconnected-(MX61-Pad2) -> COL3
- MX62 pad 1: unconnected-(MX62-Pad1) -> COL5
- MX63 pad 1: unconnected-(MX63-Pad1) -> COL7
- MX64 pad 1: unconnected-(MX64-Pad1) -> COL9
- MX65 pad 1: unconnected-(MX65-Pad1) -> COL11
- MX66 pad 1: unconnected-(MX66-Pad1) -> Net-(D65-A)
- MX66 pad 2: unconnected-(MX66-Pad2) -> COL11
- MX67 pad 1: unconnected-(MX67-Pad1) -> COL12
- MX68 pad 1: unconnected-(MX68-Pad1) -> COL13
- MX69 pad 1: unconnected-(MX69-Pad1) -> COL14
- MX7 pad 1: unconnected-(MX7-Pad1) -> COL7
- MX8 pad 1: unconnected-(MX8-Pad1) -> COL8
- MX9 pad 1: unconnected-(MX9-Pad1) -> COL9

Commit message: Complete column traces
Parts:
- Q1, Q2, R1, R2: moved to B.Cu
- moved D14 18.9 mm to (326.9, 83.9)
- moved D45 13.4 mm to (81.2, 150.2), turned to -90 degrees
- moved D60 10.5 mm to (127.2, 160.5), turned to -90 degrees
- moved D65 10.1 mm to (274.5, 160.5)
- moved D29 9.95 mm to (81.2, 122.0), turned to 180 degrees
- moved D43 7.63 mm to (73.7, 153.4), turned to 180 degrees
- moved R2 5.37 mm to (339.5, 91.9), turned to 180 degrees
- moved Q2 4.24 mm to (337.6, 95.0)
- moved R1 3.39 mm to (70.1, 90.7), turned to 180 degrees
- moved Q1 1.98 mm to (67.7, 94.6), turned to 90 degrees
Connections:
- D1 pad 1: ROW1 -> ROW0
- D10 pad 1: ROW1 -> ROW0
- D11 pad 1: ROW1 -> ROW0
- D12 pad 1: ROW1 -> ROW0
- D13 pad 1: ROW1 -> ROW0
- D14 pad 1: ROW1 -> ROW0
- D15 pad 1: ROW2 -> ROW1
- D16 pad 1: ROW2 -> ROW1
- D17 pad 1: ROW2 -> ROW1
- D18 pad 1: ROW2 -> ROW1
- D19 pad 1: ROW2 -> ROW1
- D2 pad 1: ROW1 -> ROW0
- D20 pad 1: ROW2 -> ROW1
- D21 pad 1: ROW2 -> ROW1
- D22 pad 1: ROW2 -> ROW1
- D23 pad 1: ROW2 -> ROW1
- D24 pad 1: ROW2 -> ROW1
- D25 pad 1: ROW2 -> ROW1
- D26 pad 1: ROW2 -> ROW1
- D27 pad 1: ROW2 -> ROW1
- D28 pad 1: ROW2 -> ROW1
- D29 pad 1: ROW3 -> ROW2
- D3 pad 1: ROW1 -> ROW0
- D31 pad 1: ROW3 -> ROW2
- D32 pad 1: ROW3 -> ROW2
- D33 pad 1: ROW3 -> ROW2
- D34 pad 1: ROW3 -> ROW2
- D35 pad 1: ROW3 -> ROW2
- D36 pad 1: ROW3 -> ROW2
- D37 pad 1: ROW3 -> ROW2
- D38 pad 1: ROW3 -> ROW2
- D39 pad 1: ROW3 -> ROW2
- D4 pad 1: ROW1 -> ROW0
- D40 pad 1: ROW3 -> ROW2
- D41 pad 1: ROW3 -> ROW2
- D42 pad 1: ROW3 -> ROW2
- D43 pad 1: ROW4 -> ROW3
- D45 pad 1: ROW4 -> ROW3
- D46 pad 1: ROW4 -> ROW3
- D47 pad 1: ROW4 -> ROW3
- D48 pad 1: ROW4 -> ROW3
- D49 pad 1: ROW4 -> ROW3
- D5 pad 1: ROW1 -> ROW0
- D50 pad 1: ROW4 -> ROW3
- D51 pad 1: ROW4 -> ROW3
- D52 pad 1: ROW4 -> ROW3
- D53 pad 1: ROW4 -> ROW3
- D54 pad 1: ROW4 -> ROW3
- D55 pad 1: ROW4 -> ROW3
- D56 pad 1: ROW4 -> ROW3
- D57 pad 1: ROW4 -> ROW3
- D6 pad 1: ROW1 -> ROW0
- D7 pad 1: ROW1 -> ROW0
- D8 pad 1: ROW1 -> ROW0
- D9 pad 1: ROW1 -> ROW0
- MX1 pad 1: COL1 -> COL0
- MX10 pad 1: COL10 -> COL9
- MX11 pad 1: COL11 -> COL10
- MX12 pad 1: COL12 -> COL11
- MX13 pad 1: COL13 -> COL12
- MX14 pad 1: COL14 -> COL13
- MX15 pad 1: COL1 -> COL0
- MX16 pad 1: COL2 -> COL1
- MX17 pad 1: COL3 -> COL2
- MX18 pad 1: COL4 -> COL3
- MX19 pad 1: COL5 -> COL4
- MX2 pad 1: COL2 -> COL1
- MX20 pad 1: COL6 -> COL5
- MX21 pad 1: COL7 -> COL6
- MX22 pad 1: COL8 -> COL7
- MX23 pad 1: COL9 -> COL8
- MX24 pad 1: COL10 -> COL9
- MX25 pad 1: COL11 -> COL10
- MX26 pad 1: COL12 -> COL11
- MX27 pad 1: COL13 -> COL12
- MX28 pad 1: COL14 -> COL13
- MX29 pad 1: COL1 -> COL0
- MX3 pad 1: COL3 -> COL2
- MX30 pad 2: COL1 -> COL0
- MX31 pad 1: COL2 -> COL1
- MX32 pad 1: COL3 -> COL2
- MX33 pad 1: COL4 -> COL3
- MX34 pad 1: COL5 -> COL4
- MX35 pad 1: COL6 -> COL5
- MX36 pad 1: COL7 -> COL6
- MX37 pad 1: COL8 -> COL7
- MX38 pad 1: COL9 -> COL8
- MX39 pad 1: COL10 -> COL9
- MX4 pad 1: COL4 -> COL3
- MX40 pad 1: COL11 -> COL10
- MX41 pad 1: COL13 -> COL12
- MX42 pad 1: COL14 -> COL13
- MX43 pad 2: COL1 -> COL0
- MX44 pad 1: COL1 -> COL0
- MX45 pad 1: COL2 -> COL1
- MX46 pad 1: COL3 -> COL2
- MX47 pad 1: COL4 -> COL3
- MX48 pad 1: COL5 -> COL4
- MX49 pad 1: COL6 -> COL5
- MX5 pad 1: COL5 -> COL4
- MX50 pad 1: COL7 -> COL6
- MX51 pad 1: COL8 -> COL7
- MX52 pad 1: COL9 -> COL8
- MX53 pad 1: COL10 -> COL9
- MX54 pad 1: COL11 -> COL10
- MX55 pad 1: COL12 -> COL11
- MX56 pad 1: COL13 -> COL12
- MX57 pad 1: COL14 -> COL13
- MX58 pad 1: COL1 -> COL0
- MX59 pad 1: COL2 -> COL1
- MX6 pad 1: COL6 -> COL5
- MX60 pad 1: COL3 -> COL2
- MX61 pad 2: COL3 -> COL2
- MX62 pad 1: COL5 -> COL4
- MX63 pad 1: COL7 -> COL6
- MX64 pad 1: COL9 -> COL8
- MX65 pad 1: COL11 -> COL10
- MX66 pad 2: COL11 -> COL10
- MX67 pad 1: COL12 -> COL11
- MX68 pad 1: COL13 -> COL12
- MX69 pad 1: COL14 -> COL13
- MX7 pad 1: COL7 -> COL6
- MX8 pad 1: COL8 -> COL7
- MX9 pad 1: COL9 -> COL8
- Q1 pad 2: Net-(D1-A) -> COL0
- Q1 pad 3: COL1 -> Net-(D1-A)
- Q2 pad 2: Net-(D14-A) -> COL13
- Q2 pad 3: COL14 -> Net-(D14-A)
- R1 pad 1: VDD -> +3V3
- R2 pad 1: VDD -> +3V3
Routing:
- net COL0: track 0.00 -> 117.4 mm
- net COL10: track 0.00 -> 103.6 mm
- net COL2: track 0.00 -> 102.1 mm
- net COL4: track 0.00 -> 95.3 mm
- net COL8: track 0.00 -> 91.4 mm
- net COL6: track 0.00 -> 90.9 mm
- net COL11: track 0.00 -> 89.9 mm
- net COL12: track 0.00 -> 89.9 mm
- net COL1: track 0.00 -> 88.9 mm
- net COL13: track 0.00 -> 84.3 mm
- net COL9: track 0.00 -> 72.3 mm
- net COL3: track 0.00 -> 70.3 mm
- net COL7: track 0.00 -> 69.8 mm
- net COL5: track 0.00 -> 69.8 mm
- net Net-(D14-A): track 0.00 -> 33.6 mm, vias 0 -> 2
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