File: cloak-xt.kicad_pcb (KiCad board)
At the start: 2 copper layers, 289.7 x 98 mm, 162 parts, among them J1 JST, Q1 Q_PMOS_GSD, Q2 Q_PMOS_GSD, U1 STM32F072CBT6, U3 XC6206PxxxMR-Regulator_Linear

Commit message: Complete initial colum,n/row traces
Parts:
- moved BOOT1 3.63 mm to (326.5, 160.9)
- moved RST1 3.63 mm to (320.5, 160.9)
- turned D65 to -90 degrees
Routing:
- net ROW4: track 0.20 -> 287.8 mm
- net ROW3: track 7.89 -> 278.7 mm, vias 0 -> 2
- net ROW1: track 0.00 -> 266.7 mm
- net ROW2: track 0.00 -> 263.9 mm
- net ROW0: track 19.0 -> 252.0 mm
- net Net-(D65-A): track 0.00 -> 15.9 mm
- net /B11: track 5.79 -> 1.34 mm
- net /B9: track 9.89 -> 5.80 mm
- net +3V3: track 66.8 -> 70.7 mm
- net BOOT0: track 25.6 -> 29.5 mm
- net /B7: track 7.33 -> 3.44 mm
- net /B1: track 3.71 -> 0.00 mm
- net /B0: track 3.70 -> 0.00 mm
- net /B8: track 7.99 -> 4.61 mm
- net GND: track 100.8 -> 104.0 mm
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
Commit message: Change switches text placement
Parts:
- moved C10 16.1 mm to (329.3, 117.6)
- moved C9 16.1 mm to (328.1, 114.1)
- moved U3 16.1 mm to (330.8, 115.1)
- moved C1 9.00 mm to (323.3, 140.0)
- moved C7 9.00 mm to (323.3, 138.7)
- moved C3 9.00 mm to (329.1, 127.8)
- moved C4 9.00 mm to (320.3, 128.0)
- moved C5 9.00 mm to (329.3, 136.5)
- moved C6 9.00 mm to (328.8, 138.0)
- moved R3 9.00 mm to (326.1, 142.3)
- moved R4 9.00 mm to (323.6, 142.3)
- moved U1 9.00 mm to (324.8, 132.3)
- moved BOOT1 8.76 mm to (327.2, 152.2)
- moved RST1 8.76 mm to (321.2, 152.2)
- moved C2 8.06 mm to (328.1, 125.2)
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Routing:
- net ENC1B: track 0.00 -> 260.4 mm, vias 0 -> 1
- net ENC1A: track 0.00 -> 258.4 mm, vias 0 -> 1
- net COL0: track 117.4 -> 366.4 mm
- net COL1: track 88.9 -> 312.6 mm
- net COL2: track 102.1 -> 307.4 mm
- net COL3: track 70.3 -> 254.3 mm
- net COL4: track 95.3 -> 270.8 mm
- net COL5: track 69.8 -> 226.2 mm
- net COL6: track 90.9 -> 227.4 mm
- net COL7: track 69.8 -> 184.6 mm
- net COL8: track 91.4 -> 186.0 mm
- net COL9: track 72.3 -> 150.6 mm
- net COL10: track 103.6 -> 158.3 mm
- net COL11: track 89.9 -> 128.4 mm
- net ROW2: track 263.9 -> 225.6 mm
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
Commit message: Complete BOOT/RST traces
Parts:
- moved BOOT1 3.90 mm to (325.0, 149.0)
- moved RST1 3.90 mm to (319.0, 149.0)
- moved J1 0.71 mm to (325.9, 94.6)
- moved C2 0.70 mm to (328.5, 125.8)
Connections:
- U1 pad 12: /A2 -> COL12
- U1 pad 13: /A3 -> COL11
- U1 pad 14: /A4 -> COL10
- U1 pad 15: /A5 -> COL9
- U1 pad 16: /A6 -> COL8
- U1 pad 17: /A7 -> COL7
- U1 pad 2: /C13 -> ROW3
- U1 pad 20: /B2 -> COL6
- U1 pad 21: /B10 -> COL5
- U1 pad 22: /B11 -> COL4
- U1 pad 25: /B12 -> COL3
- U1 pad 26: /B13 -> COL2
- U1 pad 27: /B14 -> COL1
- U1 pad 28: /B15 -> COL0
- U1 pad 3: /C14 -> ROW4
- U1 pad 30: /A9 -> ENC1A
- U1 pad 31: /A10 -> ENC1B
Routing:
- net +3V3: track 61.7 -> 353.7 mm, vias 5 -> 8
- net ROW2: track 225.6 -> 363.1 mm, vias 0 -> 4
- net ROW3: track 279.6 -> 356.0 mm, vias 0 -> 4
- net GND: track 84.4 -> 118.7 mm, vias 3 -> 4
- net D+: track 0.00 -> 31.6 mm
- net D-: track 0.00 -> 31.6 mm
- net ROW4: track 287.6 -> 318.9 mm
- net ENC1A: track 258.4 -> 286.9 mm
- net ENC1B: track 260.4 -> 288.4 mm
- net +5V: track 0.00 -> 24.3 mm, vias 0 -> 2
- net COL0: track 366.4 -> 384.3 mm
- net COL1: track 312.6 -> 329.7 mm
- net COL2: track 307.4 -> 323.8 mm
- net COL3: track 254.3 -> 270.2 mm
- net COL7: track 184.6 -> 190.7 mm
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
Commit message: Complete initial PCB
Complete PCB traces with matrix and ground planes. No GND vias yet.
Connections:
- U1 pad 19: /B1 -> COL6
- U1 pad 20: COL6 -> COL5
- U1 pad 21: COL5 -> COL4
- U1 pad 22: COL4 -> ROW1
- U1 pad 38: /A15 -> ROW2
- U1 pad 39: /B3 -> ROW0
- U1 pad 40: /B4 -> ENC2A
- U1 pad 41: /B5 -> ENC2B
- U1 pad 42: /B6 -> COL13
Routing:
- net ROW0: track 252.0 -> 325.4 mm, vias 0 -> 2
- net ENC2B: track 0.00 -> 66.9 mm, vias 0 -> 1
- net ENC2A: track 0.00 -> 62.0 mm, vias 0 -> 1
- net ROW1: track 246.9 -> 290.9 mm, vias 0 -> 3
- net +3V3: track 353.7 -> 386.3 mm, vias 8 -> 10
- net ROW2: track 363.1 -> 376.1 mm
- net COL13: track 78.0 -> 85.8 mm, vias 0 -> 1
- net /B9: track 5.80 -> 0.00 mm
- net /B8: track 4.61 -> 0.00 mm
- net /B5: track 4.21 -> 0.00 mm
- net GND: track 118.7 -> 122.3 mm, vias 4 -> 6
- net /B6: track 3.34 -> 0.00 mm
- net /B7: track 3.09 -> 0.00 mm
- net /B4: track 2.84 -> 0.00 mm
- net /F1: track 2.59 -> 0.00 mm
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- added copper zone on B.Cu, net GND
- added copper zone on F.Cu, net GND

Commit message: Add schematics for SK6812MINI-E on Capslock/Stepped
Parts:
- added C11: 100nF, Capacitor_SMD:C_0402_1005Metric, F.Cu at (37.5, 139.1)
- added C8: 100nF, Capacitor_SMD:C_0402_1005Metric, F.Cu at (37.5, 137.1)
- added LED1: SK6812MINI-E, PCM_marbastlib-various:LED_6028R, B.Cu at (63.0, 131.5)
- added LED2: SK6812MINI-E, PCM_marbastlib-various:LED_6028R, F.Cu at (40.0, 125.6)
- added R5: 470, Resistor_SMD:R_0402_1005Metric, F.Cu at (37.5, 135.1)
